Commit message: Start of solution for multiple robots in RViz

File: Dynamics/simulator_prototype/config/models/Jolner.urdf (robot description, URDF)
Before this commit: robot hil_sim, 1 links, 0 joints
Links:
- removed link hil_sim
- added link simulated_vessel; visual mesh filename=file:///home/Jolner.stl scale=0.01 0.01 0.01

File: Dynamics/simulator_prototype/config/models/Odin.urdf (robot description, URDF)
Before this commit: robot hil_sim, 1 links, 0 joints
Links:
- removed link hil_sim
- added link simulated_vessel; visual mesh filename=file:///home/OdinDecimated.stl scale=0.001 0.001 0.001
