Commit message: Fikset ctrl-c-problemet og pen cleanup ved terminering

File: Dynamics/simulator_prototype/config/models/Obstacle1.urdf (robot description, URDF)
Before this commit: robot obstacle_1, 1 links, 0 joints
Links:
- link obstacle_1: geometry visual mesh filename=file:///home/OdinDecimated.stl scale=0.0015 0.0015 0.0015
