Commit message: Bevegelige skip kan nå dynamisk opprettes i RVIZ

File: Dynamics/simulator_prototype/config/models/class_A_ship.urdf (robot description, URDF)
Before this commit: robot obstacle_3, 1 links, 0 joints
Links:
- link obstacle_3: geometry visual mesh filename=file:///home/uss_deplorables_small.stl scale=0.01 0.01 0.01

File: Dynamics/simulator_prototype/config/models/class_A_ship_uss_carrier.urdf (robot description, URDF)
Before this commit: robot obstacle_3, 1 links, 0 joints
Links:
- link obstacle_3: geometry visual mesh filename=file:///home/uss_deplorables.stl scale=0.1 0.1 0.1
